File: hardware/interface.sch (KiCad schematic (older format))
At the start: 0 parts

Commit message: WIP: schematic
Parts:
- added R3: 10k, Resistor_SMD:R_0805_2012Metric, symbol Device:R_Small
- added R4: 30k9, Resistor_SMD:R_0805_2012Metric, symbol Device:R_Small
- added U3: ADuM5211, Package_SO:SSOP-20_5.3x7.2mm_P0.65mm, symbol ADuM5211:ADuM5211
- added U4: TCAN1051HGV, Package_SO:SOIC-8_3.9x4.9mm_P1.27mm, symbol TCAN1051HGV:TCAN1051HGV
Connections:
- net labels added: +3.3V, +5V, +5VISO, CAN_Rx, CAN_Tx, GND, GNDISO
- wire segments 0 -> 13
Changed lines of the file:
@@
 $Descr A4 11693 8268
 encoding utf-8
-Sheet 1 4
+Sheet 3 5
 Title ""
 Date ""
@@
 Comment4 ""
 $EndDescr
+$Comp
+L TCAN1051HGV:TCAN1051HGV U4
+U 1 1 6125C8E2
+P 5850 2950
+F 0 "U4" H 6150 3500 50  0000 C CNN
+F 1 "TCAN1051HGV" H 6250 3400 50  0000 C CNN
+F 2 "Package_SO:SOIC-8_3.9x4.9mm_P1.27mm" H 5850 2950 50  0001 C CNN
+F 3 "" H 5850 2950 50  0001 C CNN
+	1    5850 2950
+	1    0    0    -1
+$EndComp
+$Comp
+L vref:GNDISO #PWR0126
+U 1 1 6125E02B
+P 5850 3450
+F 0 "#PWR0126" H 5850 3200 50  0001 C CNN
+F 1 "GNDISO" H 5855 3277 50  0000 C CNN
+F 2 "" H 5850 3450 50  0001 C CNN
+F 3 "" H 5850 3450 50  0001 C CNN
+	1    5850 3450
+	1    0    0    -1
+$EndComp
+$Comp
+L vref:+5VISO #PWR0127
+U 1 1 61263A9C
+P 5950 2450
+F 0 "#PWR0127" H 5950 2300 50  0001 C CNN
+F 1 "+5VISO" H 6000 2600 50  0000 C CNN
+F 2 "" H 5950 2450 50  0001 C CNN
+F 3 "" H 5950 2450 50  0001 C CNN
+	1    5950 2450
+	1    0    0    -1
+$EndComp
+$Comp
+L vref:GNDISO #PWR0128
+U 1 1 61266B61
+P 5350 3300
+F 0 "#PWR0128" H 5350 3050 50  0001 C CNN
+F 1 "GNDISO" H 5355 3127 50  0000 C CNN
+F 2 "" H 5350 3300 50  0001 C CNN
+F 3 "" H 5350 3300 50  0001 C CNN
+	1    5350 3300
+	1    0    0    -1
+$EndComp
+Wire Wire Line
+	5350 3300 5350 3200
+Wire Wire Line
+	5350 3200 5450 3200
+$Comp
+L ADuM5211:ADuM5211 U3
+U 1 1 6126D36C
+P 3800 2950
+F 0 "U3" H 4200 3500 50  0000 L CNN
+F 1 "ADuM5211" H 4200 3400 50  0000 L CNN
+F 2 "Package_SO:SSOP-20_5.3x7.2mm_P0.65mm" H 3800 2000 50  0001 C CIN
+F 3 "https://www.analog.com/media/en/technical-documentation/data-sheets/ADuM5210_5211_5212.pdf" H 3350 3150 50  0001 C CNN
+	1    3800 2950
+	1    0    0    -1
+$EndComp
+Wire Wire Line
+	4300 3000 5450 3000
+Wire Wire Line
+	5450 2900 4300 2900
+$Comp
+L power:+3.3V #PWR0129
+U 1 1 612755F4
+P 3650 2450
+F 0 "#PWR0129" H 3650 2300 50  0001 C CNN
+F 1 "+3.3V" H 3700 2600 50  0000 C CNN
+F 2 "" H 3650 2450 50  0001 C CNN
+F 3 "" H 3650 2450 50  0001 C CNN
+	1    3650 2450
+	1    0    0    -1
+$EndComp
+$Comp
+L power:+5V #PWR0130
+U 1 1 61275ECD
+P 3550 2450
+F 0 "#PWR0130" H 3550 2300 50  0001 C CNN
+F 1 "+5V" H 3500 2600 50  0000 C CNN
+F 2 "" H 3550 2450 50  0001 C CNN
+F 3 "" H 3550 2450 50  0001 C CNN
+	1    3550 2450
+	1    0    0    -1
+$EndComp
+$Comp
+L power:GND #PWR0131
+U 1 1 612764DF
+P 3650 3450
+F 0 "#PWR0131" H 3650 3200 50  0001 C CNN
+F 1 "GND" H 3655 3277 50  0000 C CNN
+F 2 "" H 3650 3450 50  0001 C CNN
+F 3 "" H 3650 3450 50  0001 C CNN
+	1    3650 3450
+	1    0    0    -1
+$EndComp
+$Comp
+L vref:GNDISO #PWR0132
+U 1 1 61276948
+P 3950 3450
+F 0 "#PWR0132" H 3950 3200 50  0001 C CNN
+F 1 "GNDISO" H 3955 3277 50  0000 C CNN
+F 2 "" H 3950 3450 50  0001 C CNN
+F 3 "" H 3950 3450 50  0001 C CNN
+	1    3950 3450
+	1    0    0    -1
+$EndComp
+$Comp
+L vref:+5VISO #PWR0133
+U 1 1 612769DC
+P 5750 2450
+F 0 "#PWR0133" H 5750 2300 50  0001 C CNN
+F 1 "+5VISO" H 5700 2600 50  0000 C CNN
+F 2 "" H 5750 2450 50  0001 C CNN
+F 3 "" H 5750 2450 50  0001 C CNN
+	1    5750 2450
+	1    0    0    -1
+$EndComp
+$Comp
+L vref:+5VISO #PWR0134
+U 1 1 61276C75
+P 4050 2450
+F 0 "#PWR0134" H 4050 2300 50  0001 C CNN
+F 1 "+5VISO" H 4050 2600 50  0000 C CNN
+F 2 "" H 4050 2450 50  0001 C CNN
+F 3 "" H 4050 2450 50  0001 C CNN
+	1    4050 2450
+	1    0    0    -1
+$EndComp
+Wire Wire Line
+	4050 2450 3950 2450
+Connection ~ 4050 2450
+$Comp
+L power:GND #PWR0135
+U 1 1 61277C24
+P 3200 3300
+F 0 "#PWR0135" H 3200 3050 50  0001 C CNN
+F 1 "GND" H 3205 3127 50  0000 C CNN
+F 2 "" H 3200 3300 50  0001 C CNN
+F 3 "" H 3200 3300 50  0001 C CNN
+	1    3200 3300
+	1    0    0    -1
+$EndComp
+Wire Wire Line
+	3200 3300 3200 3200
+Wire Wire Line
+	3200 3200 3300 3200
+$Comp
+L Device:R_Small R3
+U 1 1 61278725
+P 4500 3350
+F 0 "R3" V 4400 3350 50  0000 C CNN
+F 1 "10k" V 4600 3350 50  0000 C CNN
+F 2 "Resistor_SMD:R_0805_2012Metric" H 4500 3350 50  0001 C CNN
+F 3 "~" H 4500 3350 50  0001 C CNN
+	1    4500 3350
+	0    1    1    0
+$EndComp
+$Comp
+L Device:R_Small R4
+U 1 1 6127A048
+P 4700 3350
+F 0 "R4" V 4600 3350 50  0000 C CNN
+F 1 "30k9" V 4800 3350 50  0000 C CNN
+F 2 "Resistor_SMD:R_0805_2012Metric" H 4700 3350 50  0001 C CNN
+F 3 "~" H 4700 3350 50  0001 C CNN
+	1    4700 3350
+	0    1    1    0
+$EndComp
+Wire Wire Line
+	4300 3450 4300 3350
+Wire Wire Line
+	4300 3350 4400 3350
+Wire Wire Line
+	4600 3350 4600 3200
+Wire Wire Line
+	4600 3200 4300 3200
+Connection ~ 4600 3350
+$Comp
+L vref:+5VISO #PWR0136
+U 1 1 6127E1EE
+P 4900 3250
+F 0 "#PWR0136" H 4900 3100 50  0001 C CNN
+F 1 "+5VISO" H 4900 3400 50  0000 C CNN
+F 2 "" H 4900 3250 50  0001 C CNN
+F 3 "" H 4900 3250 50  0001 C CNN
+	1    4900 3250
+	1    0    0    -1
+$EndComp
+Wire Wire Line
+	4900 3250 4900 3350
+Wire Wire Line
+	4900 3350 4800 3350
+$Comp
+L vref:GNDISO #PWR0137
+U 1 1 6127C928
+P 4300 3450
+F 0 "#PWR0137" H 4300 3200 50  0001 C CNN
+F 1 "GNDISO" H 4305 3277 50  0000 C CNN
+F 2 "" H 4300 3450 50  0001 C CNN
+F 3 "" H 4300 3450 50  0001 C CNN
+	1    4300 3450
+	1    0    0    -1
+$EndComp
+Text HLabel 3300 2900 0    50   Input ~ 0
+CAN_Tx
+Text HLabel 3300 3000 0    50   Output ~ 0
+CAN_Rx
 $EndSCHEMATC
