File: hardware/power.sch (KiCad schematic (older format))
At the start: 0 parts

Commit message: WIP: schematic
Parts:
- added C1: 100n, Capacitor_SMD:C_0805_2012Metric, symbol Device:C_Small
- added C2: 2u2, Capacitor_SMD:C_0805_2012Metric, symbol Device:C_Small
- added C3: 22u, Capacitor_SMD:C_0805_2012Metric, symbol Device:C_Small
- added C4, C5: 10u, Capacitor_SMD:C_0805_2012Metric, symbol Device:C_Small
- added L1: 15u, Inductor_SMD:L_Taiyo-Yuden_NR-60xx, symbol Device:L
- added R1: 88k7, Resistor_SMD:R_0805_2012Metric, symbol Device:R_Small
- added R2: 22k1, Resistor_SMD:R_0805_2012Metric, symbol Device:R_Small
- added U1: PLMR50410XDBVR, Package_TO_SOT_SMD:SOT-23-6, symbol LMR50410:PLMR50410XDBVR
- added U2: NCP1117-3.3_SOT223, Package_TO_SOT_SMD:SOT-223-3_TabPin2, symbol Regulator_Linear:NCP1117-3.3_SOT223
Connections:
- net labels added: 24V, 3.3V, 5V, Field24V, FieldGND, GND
- wire segments 0 -> 32
