File: hardware/power.sch (KiCad schematic (older format))
At the start: 10 parts, among them U1 PLMR50410XDBVR, U2 NCP1117-3.3_SOT223

Commit message: WIP: schematic
Parts:
- added D? (x2): D, symbol Device:D
- added D?: 10V, symbol Device:D_Zener
- added D?: SMCJ26CA, symbol Device:D_TVS
- added F?: 200mA, symbol Device:Polyfuse
- added F? (x2): 200mA, symbol Device:Fuse
- added FB?: 1k@100MHz, symbol Device:Ferrite_Bead
- added Q?: Si3129DV, Package_SO:TSOP-6_1.65x3.05mm_P0.95mm, symbol Si3129DV:Si3129DV
- added R?: 10k, symbol Device:R
- added R?: 68k, symbol Device:R
- added RV?: 60V, symbol Device:Varistor
- U1: value PLMR50410XDBVR -> LMR50410
Connections:
- net labels added: VBUS
- wire segments 32 -> 55
Other:
- moved on the sheet: C1, C2, C3, C4, C5, L1, R1, R2, U2

Commit message: Power looks nice
Parts:
- removed C1: 100n, Capacitor_SMD:C_0805_2012Metric, symbol Device:C_Small
- removed C2: 2u2, Capacitor_SMD:C_0805_2012Metric, symbol Device:C_Small
- removed C3: 22u, Capacitor_SMD:C_0805_2012Metric, symbol Device:C_Small
- removed D?: D, symbol Device:D
- removed L1: 15u, Inductor_SMD:L_Taiyo-Yuden_NR-60xx, symbol Device:L
- removed R1: 88k7, Resistor_SMD:R_0805_2012Metric, symbol Device:R_Small
- removed R2: 22k1, Resistor_SMD:R_0805_2012Metric, symbol Device:R_Small
- removed U1: LMR50410, Package_TO_SOT_SMD:SOT-23-6, symbol LMR50410:PLMR50410XDBVR
- added C? (x2): 100n, symbol Device:C_Small
- added C? (x2): 68u, symbol Device:CP_Small
- added D?: 50SQ100, symbol Device:D_Schottky_Small
- added D?: D, symbol Device:D
- added L?: 100u, symbol Device:L
- added R?: 1M, symbol Device:R_Small
- added R?: 384k, symbol Device:R_Small
- added U?: MAX5035BUSA, Package_SO:SOIC-8_3.9x4.9mm_P1.27mm, symbol Regulator_Switching:MAX5035BUSA
Connections:
- wire segments 55 -> 56
Other:
- note added: "24V -> 5V"
- note added: "5V -> 3.3V"
- note added: "Power protection"
- note added: "Resettable\npolyfuse"
- note added: "Socketed fuses"
- moved on the sheet: C4, C5, D?, F?, FB?, Q?, R?, RV?, U2

Commit message: things changed
Parts:
- removed D? (x2): D, symbol Device:D
- added D4, D5: D_Schottky, Diode_SMD:D_SMA, symbol Device:D_Schottky
- C2, C3: renamed from C?; footprint (none) -> Capacitor_SMD:C_0805_2012Metric
- D1: renamed from D?; footprint (none) -> Diode_SMD:D_MiniMELF
- D2: renamed from D?; footprint (none) -> Diode_SMD:D_SMC
- R1: renamed from R?; value 68k -> 47k
- R3: renamed from R?; value 1M -> 47k
- R4: renamed from R?; value 384k -> 10k
- gave numbers to parts that had none: 12
- renumbered C4 to C5, C5 to C6
Other:
- note added: "Allowed range:\n10.5 V - 76 V"

Commit message: Changed power again
Parts:
- removed C1, C4: 68u, symbol Device:CP_Small
- removed D3: 50SQ100, symbol Device:D_Schottky_Small
- removed D4, D5: D_Schottky, Diode_SMD:D_SMA, symbol Device:D_Schottky
- removed L1: 100u, symbol Device:L
- removed R3: 47k, symbol Device:R_Small
- removed R4: 10k, symbol Device:R_Small
- removed U1: MAX5035BUSA, Package_SO:SOIC-8_3.9x4.9mm_P1.27mm, symbol Regulator_Switching:MAX5035BUSA
- removed U2: NCP1117-3.3_SOT223, Package_TO_SOT_SMD:SOT-223-3_TabPin2, symbol Regulator_Linear:NCP1117-3.3_SOT223
- added C1: 2n7, Capacitor_SMD:C_0805_2012Metric, symbol Device:C_Small
- added C19, C20: 3n3, Capacitor_SMD:C_0805_2012Metric, symbol Device:C_Small
- added C21, C22, C25, C26: 1u, Capacitor_SMD:C_0805_2012Metric, symbol Device:C_Small
- added C23: 10u, Capacitor_SMD:C_0805_2012Metric, symbol Device:C_Small
- added C24: 22u, Capacitor_SMD:C_0805_2012Metric, symbol Device:C_Small
- added C4: 22p, Capacitor_SMD:C_0805_2012Metric, symbol Device:C_Small
- added L1: 22u, symbol Device:L_Small
- added L2: 15u, symbol Device:L_Small
- added Q3: Si1967DH, Package_TO_SOT_SMD:SOT-363_SC-70-6_Handsoldering, symbol Device:Q_DUAL_PMOS_S1G1D2S2G2D1
- added R10: 14k, Resistor_SMD:R_0805_2012Metric, symbol Device:R_Small
- added R11: 19k1, Resistor_SMD:R_0805_2012Metric, symbol Device:R_Small
- added R12: 82k5, Resistor_SMD:R_0805_2012Metric, symbol Device:R_Small
- added R13: 18k2, Resistor_SMD:R_0805_2012Metric, symbol Device:R_Small
- added R14: 54k9, Resistor_SMD:R_0805_2012Metric, symbol Device:R_Small
- added R15: 20k5, Resistor_SMD:R_0805_2012Metric, symbol Device:R_Small
- added R16, R17: 10k, Resistor_SMD:R_0805_2012Metric, symbol Device:R_Small
- added R3: 68k, Resistor_SMD:R_0805_2012Metric, symbol Device:R
- added R4: 10k, Resistor_SMD:R_0805_2012Metric, symbol Device:R
- added U1: MAX17521, MAX17521:QFN50P500X400X80-25N, symbol MAX17521ATG_:MAX17521
- added U2: AP2139AK-3.3, Package_TO_SOT_SMD:SOT-23-5, symbol Regulator_Linear:AP2127K-3.3
- C2: value 100n -> 2n7
- C3: value 100n -> 33p
- C5, C6: value 10u -> 2u2
- FB1: footprint (none) -> Inductor_SMD:L_0805_2012Metric
- R1: value 47k -> 68k; footprint (none) -> Resistor_SMD:R_0805_2012Metric
- R2: footprint (none) -> Resistor_SMD:R_0805_2012Metric
- RV1: value 60V -> MOV-10D680K; footprint (none) -> Varistor:RV_Disc_D12mm_W4.4mm_P7.5mm
Connections:
- net 24V: now also C5.1, C6.1, R3.1, U1.18 (VIN2), U1.2 (VIN1)
- net 3.3V: now also C24.1, L2.2, Q3.3 (D), R14.1; no longer C6.1
- net 5V: now also C23.1, L1.2, Q3.5 (G), R12.1, R17.1
- net GND: now also C3.2, C1.2, C19.2, C20.2, C21.1, C22.1, C23.2, C24.2, C25.2, C26.2, C4.2, R13.2, R15.2, R16.2, R17.2, R4.2, U1.1 (PGND1), U1.13 (SGND2), U1.19 (PGND2), U1.25 (EXP), U1.7 (SGND1), U2.2 (GND)
- net at C3.1: now also R10.1, U1.8 (COMP1)
- net at C2.1: now also R11.2
- net at F3.1: now also C25.1, U2.1 (VIN), U2.3 (EN)
- new net: C4.1, R11.1, U1.12 (COMP2)
- new net: C20.1, U1.14 (SS2)
- new net: R14.2, R15.1, U1.15 (FB2)
- new net: C22.2, U1.16 (VCC2)
- new net: R3.2, R4.1, U1.17 (EN/UVLO2), U1.3 (EN/UVLO1)
- new net: L2.1, U1.20 (LX2)
- new net: L1.1, U1.24 (LX1)
- new net: C21.2, U1.4 (VCC1)
- new net: R12.2, R13.1, U1.5 (FB1)
- new net: C19.1, U1.6 (SS1)
- new net: C1.1, R10.2
- new net: C26.1, Q3.4 (S), R16.1, U2.5 (VOUT)
- new net PG3V3: U1.11 (~RESET2)
- new net PG5V: U1.9 (~RESET1)
- no-connect marks 0 -> 4
Other:
- note added: "3.3V, 5V"
- note added: "Allowed range:\n9.5V - 60V"
- note added: "USB 3.3V"
- note removed: "24V -> 5V"
- note removed: "5V -> 3.3V"
- note removed: "Allowed range:\n10.5 V - 76 V"
- moved on the sheet: D1, D2, F1, F2, F3, FB1, Q1, R1, R2, RV1

Commit message: Started routing
Parts:
- D2: value SMCJ26CA -> SMAJ26CA; footprint Diode_SMD:D_SMC -> Diode_SMD:D_SMA
- F1, F2: value 200mA -> 500mA; footprint (none) -> Littelfuse-154:Littelfuse-154
- F3: value 200mA -> 500mA; footprint (none) -> Fuse:Fuse_1206_3216Metric
- L1: footprint (none) -> Inductor_SMD:L_Taiyo-Yuden_NR-80xx_HandSoldering; PartNo (none) -> TaiyoYuden NRS8040T220MJGJ
- L2: footprint (none) -> Inductor_SMD:L_Taiyo-Yuden_NR-80xx_HandSoldering; PartNo (none) -> TaiyoYuden NRS8040T150MJGJ
Connections:
- net FSEL: now reaches U1.10 (FSEL)
- net COMP2: now reaches C4.1, R11.1, U1.12 (COMP2)
- net SS2: now reaches C20.1, U1.14 (SS2)
- net FB2: now reaches R14.2, R15.1, U1.15 (FB2)
- net VCC2: now reaches C22.2, U1.16 (VCC2)
- net UVLO: now reaches R3.2, R4.1, U1.17 (EN/UVLO2), U1.3 (EN/UVLO1)
- net LX2: now reaches L2.1, U1.20 (LX2)
- net MODE2: now reaches U1.21 (MODE2)
- net SYNC: now reaches U1.22 (SYNC)
- net MODE1: now reaches U1.23 (MODE1)
- net LX1: now reaches L1.1, U1.24 (LX1)
- net VCC1: now reaches C21.2, U1.4 (VCC1)
- net FB1: now reaches R12.2, R13.1, U1.5 (FB1)
- net SS1: now reaches C19.1, U1.6 (SS1)
- net COMP1: now reaches C3.1, R10.1, U1.8 (COMP1)
Other:
- note added: "PPTC fuse\nBelFuse 0ZCJ0025FF2E"
- note added: "Socketed fuses\nLittelfuse 154"
- note removed: "Resettable\npolyfuse"
- note removed: "Socketed fuses"
- moved on the sheet: C21, C22
Changed lines of the file:
@@
 P 1700 1350
 F 0 "F1" V 1600 1200 50  0000 C CNN
-F 1 "200mA" V 1600 1500 50  0000 C CNN
-F 2 "" V 1630 1350 50  0001 C CNN
-F 3 "~" H 1700 1350 50  0001 C CNN
+F 1 "500mA" V 1600 1500 50  0000 C CNN
+F 2 "Littelfuse-154:Littelfuse-154" V 1630 1350 50  0001 C CNN
+F 3 "https://hu.mouser.com/datasheet/2/240/Littelfuse_Fuse_154_154T_154L_154TL_Datasheet_pdf-365375.pdf" H 1700 1350 50  0001 C CNN
 	1    1700 1350
-	0    1    1    0
-$EndComp
-$Comp
-L Device:Fuse F2
-U 1 1 61283881
-P 1700 1950
-F 0 "F2" V 1600 1800 50  0000 C CNN
-F 1 "200mA" V 1600 2100 50  0000 C CNN
-F 2 "" V 1630 1950 50  0001 C CNN
-F 3 "~" H 1700 1950 50  0001 C CNN
-	1    1700 1950
 	0    1    1    0
 $EndComp
@@
 P 4150 1650
 F 0 "D2" V 4104 1730 50  0000 L CNN
-F 1 "SMCJ26CA" V 4195 1730 50  0000 L CNN
-F 2 "Diode_SMD:D_SMC" H 4150 1650 50  0001 C CNN
+F 1 "SMAJ26CA" V 4195 1730 50  0000 L CNN
+F 2 "Diode_SMD:D_SMA" H 4150 1650 50  0001 C CNN
 F 3 "~" H 4150 1650 50  0001 C CNN
 	1    4150 1650
@@
 Power protection
 Text Notes 1450 2150 0    50   ~ 0
-Socketed fuses
+Socketed fuses\nLittelfuse 154
 $Comp
 L Device:Q_DUAL_PMOS_S1G1D2S2G2D1 Q3
@@
 L power:GND #PWR013
 U 1 1 614A2B10
-P 4900 6250
-F 0 "#PWR013" H 4900 6000 50  0001 C CNN
-F 1 "GND" H 4900 6100 50  0000 C CNN
-F 2 "" H 4900 6250 50  0001 C CNN
-F 3 "" H 4900 6250 50  0001 C CNN
-	1    4900 6250
+P 5000 6250
+F 0 "#PWR013" H 5000 6000 50  0001 C CNN
+F 1 "GND" H 5000 6100 50  0000 C CNN
+F 2 "" H 5000 6250 50  0001 C CNN
+F 3 "" H 5000 6250 50  0001 C CNN
+	1    5000 6250
 	1    0    0    -1
 $EndComp
@@
 L vref:PGND #PWR017
 U 1 1 614AFB99
-P 5100 6250
-F 0 "#PWR017" H 5100 6000 50  0001 C CNN
-F 1 "PGND" H 5100 6100 50  0000 C CNN
-F 2 "" H 5100 6250 50  0001 C CNN
-F 3 "" H 5100 6250 50  0001 C CNN
-	1    5100 6250
-	1    0    0    -1
-$EndComp
-Wire Wire Line
-	5100 6250 5100 6150
-Wire Wire Line
-	5100 6150 4900 6150
-Wire Wire Line
-	4900 6250 4900 6150
+P 5200 6250
+F 0 "#PWR017" H 5200 6000 50  0001 C CNN
+F 1 "PGND" H 5200 6100 50  0000 C CNN
+F 2 "" H 5200 6250 50  0001 C CNN
+F 3 "" H 5200 6250 50  0001 C CNN
+	1    5200 6250
+	1    0    0    -1
+$EndComp
+Wire Wire Line
+	5200 6250 5200 6150
+Wire Wire Line
+	5200 6150 5000 6150
+Wire Wire Line
+	5000 6250 5000 6150
 $Comp
 L power:GND #PWR012
@@
 	1    0    0    -1
 $EndComp
-$Comp
-L Device:L_Small L2
-U 1 1 614D8627
-P 4800 4750
-F 0 "L2" V 4850 4850 50  0000 C CNN
-F 1 "15u" V 4850 4650 50  0000 C CNN
-F 2 "" H 4800 4750 50  0001 C CNN
-F 3 "~" H 4800 4750 50  0001 C CNN
-	1    4800 4750
-	0    -1   -1   0
-$EndComp
 Wire Wire Line
 	4500 4150 5000 4150
@@
 F 0 "L1" V 4850 4050 50  0000 C CNN
 F 1 "22u" V 4850 3850 50  0000 C CNN
-F 2 "" H 4800 3950 50  0001 C CNN
-F 3 "~" H 4800 3950 50  0001 C CNN
+F 2 "Inductor_SMD:L_Taiyo-Yuden_NR-80xx_HandSoldering" H 4800 3950 50  0001 C CNN
+F 3 "https://hu.mouser.com/datasheet/2/396/wound04_e-1290968.pdf" H 4800 3950 50  0001 C CNN
+F 4 "TaiyoYuden NRS8040T220MJGJ" V 4800 3950 50  0001 C CNN "PartNo"
 	1    4800 3950
 	0    -1   -1   0
 $EndComp
 Wire Wire Line
-	4900 6150 4900 5950
-Connection ~ 4900 6150
-Wire Wire Line
-	4800 6150 4900 6150
-Wire Wire Line
-	4900 5950 4800 5950
-Wire Wire Line
-	4600 6150 4500 6150
-Wire Wire Line
-	4500 5950 4600 5950
+	5000 6150 5000 5950
+Connection ~ 5000 6150
+Wire Wire Line
+	4900 6150 5000 6150
+Wire Wire Line
+	5000 5950 4900 5950
 $Comp
 L Device:C_Small C22
 U 1 1 614965C6
-P 4700 6150
-F 0 "C22" V 4600 6050 50  0000 C CNN
-F 1 "1u" V 4600 6250 50  0000 C CNN
-F 2 "Capacitor_SMD:C_0805_2012Metric" H 4700 6150 50  0001 C CNN
-F 3 "~" H 4700 6150 50  0001 C CNN
-	1    4700 6150
+P 4800 6150
+F 0 "C22" V 4700 6050 50  0000 C CNN
+F 1 "1u" V 4700 6250 50  0000 C CNN
+F 2 "Capacitor_SMD:C_0805_2012Metric" H 4800 6150 50  0001 C CNN
+F 3 "~" H 4800 6150 50  0001 C CNN
+	1    4800 6150
 	0    1    1    0
 $EndComp
@@
 L Device:C_Small C21
 U 1 1 61495E1E
-P 4700 5950
-F 0 "C21" V 4600 5850 50  0000 C CNN
-F 1 "1u" V 4600 6050 50  0000 C CNN
-F 2 "Capacitor_SMD:C_0805_2012Metric" H 4700 5950 50  0001 C CNN
-F 3 "~" H 4700 5950 50  0001 C CNN
-	1    4700 5950
+P 4800 5950
+F 0 "C21" V 4700 5850 50  0000 C CNN
+F 1 "1u" V 4700 6050 50  0000 C CNN
+F 2 "Capacitor_SMD:C_0805_2012Metric" H 4800 5950 50  0001 C CNN
+F 3 "~" H 4800 5950 50  0001 C CNN
+	1    4800 5950
 	0    1    1    0
 $EndComp
@@
 NoConn ~ 3000 4450
 NoConn ~ 3000 4350
-$Comp
-L MAX17521ATG_:MAX17521 U1
-U 1 1 61419DB0
-P 3750 5250
-F 0 "U1" H 4400 6900 50  0000 C CNN
-F 1 "MAX17521" H 3750 6900 50  0000 C CNN
-F 2 "MAX17521:QFN50P500X400X80-25N" H 3100 6400 50  0001 C CNN
-F 3 "https://datasheets.maximintegrated.com/en/ds/MAX17521.pdf" H 3100 6400 50  0001 C CNN
-	1    3750 5250
-	1    0    0    -1
-$EndComp
 Text Notes 700  3550 0    100  ~ 20
 3.3V, 5V
@@
 	1    0    0    -1
 $EndComp
-Text Notes 7000 1500 0    50   ~ 0
-Resettable\npolyfuse
+Text Notes 7150 1300 0    50   ~ 0
+PPTC fuse\nBelFuse 0ZCJ0025FF2E
 Wire Wire Line
 	7750 1600 7650 1600
@@
 P 7500 1600
 F 0 "F3" V 7300 1600 50  0000 C CNN
-F 1 "200mA" V 7400 1600 50  0000 C CNN
-F 2 "" H 7550 1400 50  0001 L CNN
-F 3 "~" H 7500 1600 50  0001 C CNN
+F 1 "500mA" V 7400 1600 50  0000 C CNN
+F 2 "Fuse:Fuse_1206_3216Metric" H 7550 1400 50  0001 L CNN
+F 3 "https://www.belfuse.com/resources/datasheets/circuitprotection/ds-cp-0zcj-series.pdf" H 7500 1600 50  0001 C CNN
 	1    7500 1600
 	0    1    1    0
@@
 Wire Wire Line
 	6850 1600 7350 1600
+$Comp
+L Device:L_Small L2
+U 1 1 61247B76
+P 4800 4750
+F 0 "L2" V 4850 4850 50  0000 C CNN
+F 1 "15u" V 4850 4650 50  0000 C CNN
+F 2 "Inductor_SMD:L_Taiyo-Yuden_NR-80xx_HandSoldering" H 4800 4750 50  0001 C CNN
+F 3 "https://hu.mouser.com/datasheet/2/396/wound04_e-1290968.pdf" H 4800 4750 50  0001 C CNN
+F 4 "TaiyoYuden NRS8040T150MJGJ" V 4800 4750 50  0001 C CNN "PartNo"
+	1    4800 4750
+	0    -1   -1   0
+$EndComp
+$Comp
+L Device:Fuse F2
+U 1 1 6124AA85
+P 1700 1950
+F 0 "F2" V 1600 1800 50  0000 C CNN
+F 1 "500mA" V 1600 2100 50  0000 C CNN
+F 2 "Littelfuse-154:Littelfuse-154" V 1630 1950 50  0001 C CNN
+F 3 "https://hu.mouser.com/datasheet/2/240/Littelfuse_Fuse_154_154T_154L_154TL_Datasheet_pdf-365375.pdf" H 1700 1950 50  0001 C CNN
+	1    1700 1950
+	0    1    1    0
+$EndComp
+Text Label 4500 3950 0    50   ~ 0
+LX1
+Text Label 4500 4150 0    50   ~ 0
+FB1
+Text Label 4500 4750 0    50   ~ 0
+LX2
+Text Label 4500 4950 0    50   ~ 0
+FB2
+Text Label 4500 5950 0    50   ~ 0
+VCC1
+Text Label 4500 6150 0    50   ~ 0
+VCC2
+Wire Wire Line
+	4500 5950 4700 5950
+Wire Wire Line
+	4500 6150 4700 6150
+Text Label 3000 6050 2    50   ~ 0
+COMP1
+Text Label 3000 6550 2    50   ~ 0
+COMP2
+$Comp
+L MAX17521ATG_:MAX17521 U1
+U 1 1 61419DB0
+P 3750 5250
+F 0 "U1" H 4400 6900 50  0000 C CNN
+F 1 "MAX17521" H 3750 6900 50  0000 C CNN
+F 2 "MAX17521:QFN50P500X400X80-25N" H 3100 6400 50  0001 C CNN
+F 3 "https://datasheets.maximintegrated.com/en/ds/MAX17521.pdf" H 3100 6400 50  0001 C CNN
+	1    3750 5250
+	1    0    0    -1
+$EndComp
+Text Label 3000 5450 2    50   ~ 0
+SS1
+Text Label 3000 5650 2    50   ~ 0
+SS2
+Text Label 2900 5050 2    50   ~ 0
+UVLO
+Text Label 3000 4350 2    50   ~ 0
+FSEL
+Text Label 3000 4450 2    50   ~ 0
+SYNC
+Text Label 3000 4650 2    50   ~ 0
+MODE1
+Text Label 3000 4750 2    50   ~ 0
+MODE2
 $EndSCHEMATC
