File: hardware/hardware.kicad_pcb (KiCad board)
At the start: 2 copper layers, 333.4 x 239.8 mm, 91 parts, among them J1 USB_C_Receptacle_USB2.0, J2 Conn_ST_STDC14, J3 Micro_SD_Card_Det, J4 RJHSE5380, J5 RJHSE5380, J6 OQ0271010000G, J7 OQ0271010000G, J8 Conn_02x13_Odd_Even_MountingP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, Q1 Si3129DV, Q2 PMDT290UNE, Q3 Si1967DH, SW1 218-8LPS, SW2 Boot0, SW3 User, SW4 nReset, U1 MAX17521, U2 AP2139AK-3.3, U3 USBLC6-4SC6, U4 TCAN1051HGV, U5 STM32G474VET6, Y1 25MHz

Commit message: things changed
Parts:
- removed D6, D7: TBU-CA040-200-WH, TBU-CA:DIOC650X400X100N
- moved C12 52.1 mm to (170.9, 116.1), turned to 90 degrees
- moved C9 44.9 mm to (174.8, 112.8), turned to 180 degrees
- moved J1 38.0 mm to (90.8, 166.5)
- moved Y1 37.1 mm to (174.8, 116.1), turned to 180 degrees
- moved J2 28.6 mm to (228.1, 103.0)
- moved JP4 20.1 mm to (33.5, 130.4)
- moved C28 12.8 mm to (50.9, 142.0)
- moved C27 12.8 mm to (50.9, 146.1)
- moved U4 12.8 mm to (46.9, 144.0)
- moved D8 9.92 mm to (46.9, 136.7)
- moved SW1 7.73 mm to (175.3, 124.7), turned to 90 degrees
- moved RN2 5.73 mm to (258.9, 114.0)
- moved LD1 5.73 mm to (255.5, 126.0)
- moved Q2 5.73 mm to (255.8, 114.0)
- moved RN1 5.73 mm to (252.1, 114.0)
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Connections:
- J4 pad 4: /interface/CANL -> Net-(J4-Pad4)
- J4 pad 5: /interface/CANH -> Net-(J4-Pad5)
- J4 pad 7: Net-(J4-Pad7) -> /interface/CANL
- J4 pad 8: Net-(J4-Pad8) -> /interface/CANH
- J5 pad 4: /interface/CANL -> Net-(J4-Pad4)
- J5 pad 5: /interface/CANH -> Net-(J4-Pad5)
- J5 pad 7: Net-(J4-Pad7) -> /interface/CANL
- J5 pad 8: Net-(J4-Pad8) -> /interface/CANH
- U4 pad 6: Net-(D7-Pad1) -> /interface/CANL
- U4 pad 7: Net-(D6-Pad1) -> /interface/CANH
Routing:
- net /interface/CANL: track 0.00 -> 53.6 mm, vias 0 -> 2
- net Net-(J4-PadSH): track 0.00 -> 45.7 mm
- net /interface/CANH: track 0.00 -> 40.9 mm, vias 0 -> 2
- net /interface/RX+: track 0.00 -> 33.9 mm, vias 0 -> 2
- net Net-(J4-Pad5): track 0.00 -> 32.9 mm, vias 0 -> 2
- net /interface/RX-: track 0.00 -> 32.5 mm, vias 0 -> 2
- net Net-(J4-Pad4): track 0.00 -> 30.9 mm, vias 0 -> 2
- net /interface/TX+: track 0.00 -> 30.6 mm, vias 0 -> 2
- net /interface/TX-: track 0.00 -> 29.6 mm, vias 0 -> 2
- net +24V: track 19.6 -> 43.1 mm, vias 2 -> 3
- net /mcu/OscOut: track 0.00 -> 16.0 mm
- net /mcu/OscIn: track 0.00 -> 13.7 mm
- net +5V: track 0.00 -> 9.75 mm, vias 6 -> 5
- net +3V3: track 0.00 -> 8.89 mm, vias 6 -> 5
- net GND: vias 22 -> 26
- added copper zone on F.Cu, net GND
Other:
- board size 333.4 x 239.8 mm -> 85.9 x 116.5 mm
- rule trace_min: 0.2 -> 0.15
