File: hardware/mcu.sch (KiCad schematic (older format))
At the start: 16 parts

Commit message: WIP: schematic
Parts:
- removed C? (x2): TBD, symbol Device:C_Small
- removed FB?: 1k@100MHz, symbol Device:Ferrite_Bead_Small
- removed U?: STM32G474VET6, QFP50P1600X1600X160-100N, symbol STM32G474VET6:STM32G474VET6
- removed Y?: 8MHz, symbol Device:Crystal_GND24_Small
- added C16, C17: TBD, Capacitor_SMD:C_0805_2012Metric, symbol Device:C_Small
- added FB1: 1k@100MHz, Inductor_SMD:L_0805_2012Metric, symbol Device:Ferrite_Bead_Small
- added U5: STM32G474VET6, Package_QFP:TQFP-100_14x14mm_P0.5mm, symbol STM32G474VET6:STM32G474VET6
- added Y1: 25MHz, Crystal:Crystal_SMD_3225-4Pin_3.2x2.5mm_HandSoldering, symbol Device:Crystal_GND24_Small
- C10, C11, C12, C13, C14, C15, C6, C7, C8, C9: renamed from C?; footprint (none) -> Capacitor_SMD:C_0805_2012Metric
- JP1: renamed from JP?; footprint (none) -> Jumper:SolderJumper-2_P1.3mm_Bridged_RoundedPad1.0x1.5mm
Connections:
- net labels added: +VREF, Boot0, CAN_Rx, CAN_Tx, ClkOut, Dig_0, Dig_1, Heartbeat, OscIn, OscOut, SD_SPI_MISO, SD_SPI_MOSI, SD_SPI_SCK, SD_SPI_nSS, SWCLK, SWDIO, Seg_0, Seg_1, Seg_2, Seg_3, Seg_4, Seg_5, Seg_6, Seg_7, Sw_0, Sw_1, Sw_2, Sw_3, Sw_4, Sw_5, Sw_6, Sw_7, UserBtn, UserLED, dbg_UART_Rx, dbg_UART_Tx, ext_CAN_Rx, ext_CAN_Tx, ext_SPI_MISO, ext_SPI_MOSI, ext_SPI_SCK, ext_SPI_nSS, ext_UART_Rx, ext_UART_Tx, nRST
- net labels removed: NRST, VREF+
- wire segments 39 -> 64
Other:
- note added: "FDCAN1"
- note added: "FDCAN2"
- note added: "SPI1"
- note added: "SPI3"
- note added: "UART4"
- note added: "USART1"
- moved on the sheet: C10, C11, C12, C13, C14, C15, C6, C7, C8, C9, JP1

Commit message: WIP: schematic
Parts:
- added J2: Conn_ST_STDC14, symbol Connector:Conn_ST_STDC14
- C10, C6, C7, C8, C9: value 100nF -> 100n
- C11: value 4.7uF -> 4u7
- C12, C15: value 1uF -> 1u
- C13, C14: value 10nF -> 10n
Connections:
- net +3V3: now also J2.3 (VCC)
- net GND: now also J2.5 (GND), J2.7 (GND)
- net SD_SPI_MISO: now also U5.80 (PC11); no longer U5.91 (PB4)
- net SD_SPI_MOSI: now also U5.81 (PC12); no longer U5.92 (PB5)
- net SD_SPI_SCK: now also U5.79 (PC10); no longer U5.90 (PB3)
- net dbg_UART_Rx: now also U5.88 (PD6), J2.13 (VCP_RX); no longer U5.80 (PC11)
- net dbg_UART_Tx: now also U5.87 (PD5), J2.14 (VCP_TX); no longer U5.79 (PC10)
- net nRST: now also J2.12 (~RST)
- net USB_CC1: now reaches U5.93 (PB6)
- net SWCLK renamed dbg_SWCLK
- net dbg_SWCLK: now also J2.6 (JCLK/SWCLK)
- net SWDIO renamed dbg_SWDIO
- net dbg_SWDIO: now also J2.4 (JTMS/SWDIO)
- net USB+ renamed USB_D+
- net USB- renamed USB_D-
- new net USB_CC2: U5.91 (PB4)
- new net dbg_SWO: J2.8 (JTDO/SWO), U5.90 (PB3)
- no-connect marks 0 -> 3
Other:
- note added: "No external termination needed\ndatasheet p.180"
- note added: "USART2"
- note removed: "UART4"
Changed lines of the file:
@@
 P 8650 900
 F 0 "C6" H 8750 950 50  0000 L CNN
-F 1 "100nF" H 8750 850 50  0000 L CNN
+F 1 "100n" H 8750 850 50  0000 L CNN
 F 2 "Capacitor_SMD:C_0805_2012Metric" H 8650 900 50  0001 C CNN
 F 3 "~" H 8650 900 50  0001 C CNN
@@
 P 9050 900
 F 0 "C7" H 9150 950 50  0000 L CNN
-F 1 "100nF" H 9150 850 50  0000 L CNN
+F 1 "100n" H 9150 850 50  0000 L CNN
 F 2 "Capacitor_SMD:C_0805_2012Metric" H 9050 900 50  0001 C CNN
 F 3 "~" H 9050 900 50  0001 C CNN
@@
 P 9450 900
 F 0 "C8" H 9550 950 50  0000 L CNN
-F 1 "100nF" H 9550 850 50  0000 L CNN
+F 1 "100n" H 9550 850 50  0000 L CNN
 F 2 "Capacitor_SMD:C_0805_2012Metric" H 9450 900 50  0001 C CNN
 F 3 "~" H 9450 900 50  0001 C CNN
@@
 P 9850 900
 F 0 "C9" H 9950 950 50  0000 L CNN
-F 1 "100nF" H 9950 850 50  0000 L CNN
+F 1 "100n" H 9950 850 50  0000 L CNN
 F 2 "Capacitor_SMD:C_0805_2012Metric" H 9850 900 50  0001 C CNN
 F 3 "~" H 9850 900 50  0001 C CNN
@@
 P 10250 900
 F 0 "C10" H 10350 950 50  0000 L CNN
-F 1 "100nF" H 10350 850 50  0000 L CNN
+F 1 "100n" H 10350 850 50  0000 L CNN
 F 2 "Capacitor_SMD:C_0805_2012Metric" H 10250 900 50  0001 C CNN
 F 3 "~" H 10250 900 50  0001 C CNN
@@
 P 10750 900
 F 0 "C11" H 10850 950 50  0000 L CNN
-F 1 "4.7uF" H 10850 850 50  0000 L CNN
+F 1 "4u7" H 10850 850 50  0000 L CNN
 F 2 "Capacitor_SMD:C_0805_2012Metric" H 10750 900 50  0001 C CNN
 F 3 "~" H 10750 900 50  0001 C CNN
@@
 P 10750 1750
 F 0 "C15" H 10850 1800 50  0000 L CNN
-F 1 "1uF" H 10850 1700 50  0000 L CNN
+F 1 "1u" H 10850 1700 50  0000 L CNN
 F 2 "Capacitor_SMD:C_0805_2012Metric" H 10750 1750 50  0001 C CNN
 F 3 "~" H 10750 1750 50  0001 C CNN
@@
 P 10250 1750
 F 0 "C14" H 10350 1800 50  0000 L CNN
-F 1 "10nF" H 10350 1700 50  0000 L CNN
+F 1 "10n" H 10350 1700 50  0000 L CNN
 F 2 "Capacitor_SMD:C_0805_2012Metric" H 10250 1750 50  0001 C CNN
 F 3 "~" H 10250 1750 50  0001 C CNN
@@
 P 8650 1750
 F 0 "C12" H 8750 1800 50  0000 L CNN
-F 1 "1uF" H 8750 1700 50  0000 L CNN
+F 1 "1u" H 8750 1700 50  0000 L CNN
 F 2 "Capacitor_SMD:C_0805_2012Metric" H 8650 1750 50  0001 C CNN
 F 3 "~" H 8650 1750 50  0001 C CNN
@@
 P 9150 1750
 F 0 "C13" H 9250 1800 50  0000 L CNN
-F 1 "10nF" H 9250 1700 50  0000 L CNN
+F 1 "10n" H 9250 1700 50  0000 L CNN
 F 2 "Capacitor_SMD:C_0805_2012Metric" H 9150 1750 50  0001 C CNN
 F 3 "~" H 9150 1750 50  0001 C CNN
@@
 Connection ~ 9150 1850
 Text Label 1450 3000 0    50   ~ 0
-USB-
+USB_D-
 Text Label 1450 3100 0    50   ~ 0
-USB+
+USB_D+
 $Comp
 L STM32G474VET6:STM32G474VET6 U5
@@
 	1    0    0    -1
 $EndComp
-Text Label 4250 2000 2    50   ~ 0
+Text Label 4450 2000 2    50   ~ 0
 CAN_Tx
-Text Label 4250 1900 2    50   ~ 0
+Text Label 4450 1900 2    50   ~ 0
 CAN_Rx
-Wire Wire Line
-	3950 1900 4250 1900
-Wire Wire Line
-	4250 2000 3950 2000
 Text Label 1450 4900 0    50   ~ 0
 ext_CAN_Tx
@@
 ext_CAN_Rx
 Text Label 1450 3200 0    50   ~ 0
-SWDIO
+dbg_SWDIO
 Text Label 1450 3300 0    50   ~ 0
-SWCLK
+dbg_SWCLK
 $Comp
 L power:+3.3V #PWR0111
@@
 	9150 1850 10250 1850
 Connection ~ 10250 1850
-Text Label 4250 5700 2    50   ~ 0
+Text Label 4450 5700 2    50   ~ 0
 OscIn
-Text Label 4250 5800 2    50   ~ 0
+Text Label 4450 5800 2    50   ~ 0
 OscOut
-Wire Wire Line
-	4250 5700 3950 5700
-Wire Wire Line
-	3950 5800 4250 5800
 Text Label 8550 2750 0    50   ~ 0
 OscIn
@@
 	8550 2750 8850 2750
 Connection ~ 8850 2750
-Text HLabel 1850 4400 0    50   Input ~ 0
+Text HLabel 1450 4400 0    50   Input ~ 0
 Boot0
-Text HLabel 1850 2700 0    50   Output ~ 0
+Text HLabel 1450 2700 0    50   Output ~ 0
 ClkOut
-Text HLabel 1850 1700 0    50   Input ~ 0
+Text HLabel 1450 1700 0    50   Input ~ 0
 nRST
 Text Label 1450 2300 0    50   ~ 0
@@
 SPI1
 Wire Wire Line
-	1850 4400 1950 4400
-Wire Wire Line
-	1850 2700 1950 2700
-Wire Wire Line
-	1850 1700 1950 1700
-Wire Wire Line
 	1450 3300 1950 3300
 Wire Wire Line
@@
 $EndComp
 Connection ~ 8650 1650
+Text Label 4450 2400 2    50   ~ 0
+dbg_UART_Tx
+Text Label 4450 2500 2    50   ~ 0
+dbg_UART_Rx
+Wire Wire Line
+	4450 2500 3950 2500
+Wire Wire Line
+	3950 2400 4450 2400
+Text Notes 4450 2300 2    50   ~ 0
+USART2
 Text Label 1450 6300 0    50   ~ 0
-dbg_UART_Tx
+SD_SPI_SCK
 Text Label 1450 6400 0    50   ~ 0
-dbg_UART_Rx
-Wire Wire Line
-	1450 6400 1950 6400
-Wire Wire Line
-	1950 6300 1450 6300
-Text Notes 1450 6200 0    50   ~ 0
-UART4
-Text Label 1450 3900 0    50   ~ 0
-SD_SPI_SCK
-Text Label 1450 4000 0    50   ~ 0
 SD_SPI_MISO
-Text Label 1450 4100 0    50   ~ 0
+Text Label 1450 6500 0    50   ~ 0
 SD_SPI_MOSI
 Wire Wire Line
-	1450 4100 1950 4100
-Wire Wire Line
-	1950 4000 1450 4000
-Wire Wire Line
-	1450 3900 1950 3900
+	1450 6500 1950 6500
+Wire Wire Line
+	1950 6400 1450 6400
+Wire Wire Line
+	1450 6300 1950 6300
 Text Label 1450 3400 0    50   ~ 0
 SD_SPI_nSS
 Wire Wire Line
 	1450 3400 1950 3400
-Text Notes 1450 3800 0    50   ~ 0
+Text Notes 1450 6200 0    50   ~ 0
 SPI3
-Text Notes 4250 1800 2    50   ~ 0
+Text Notes 4450 1800 2    50   ~ 0
 FDCAN1
-Text HLabel 5350 1500 0    50   Output ~ 0
+Text HLabel 7400 1150 0    50   Output ~ 0
 Seg_0
-Text HLabel 5350 1600 0    50   Output ~ 0
+Text HLabel 7400 1250 0    50   Output ~ 0
 Seg_1
-Text HLabel 5350 1700 0    50   Output ~ 0
+Text HLabel 7400 1350 0    50   Output ~ 0
 Seg_2
-Text HLabel 5350 1800 0    50   Output ~ 0
+Text HLabel 7400 1450 0    50   Output ~ 0
 Seg_3
-Text HLabel 5350 1900 0    50   Output ~ 0
+Text HLabel 7400 1550 0    50   Output ~ 0
 Seg_4
-Text HLabel 5350 2000 0    50   Output ~ 0
+Text HLabel 7400 1650 0    50   Output ~ 0
 Seg_5
-Text HLabel 5350 2100 0    50   Output ~ 0
+Text HLabel 7400 1750 0    50   Output ~ 0
 Seg_6
-Text HLabel 5350 2200 0    50   Output ~ 0
+Text HLabel 7400 1850 0    50   Output ~ 0
 Seg_7
-Text HLabel 5350 2300 0    50   Output ~ 0
+Text HLabel 7400 1950 0    50   Output ~ 0
 Dig_0
-Text HLabel 5350 2400 0    50   Output ~ 0
+Text HLabel 7400 2050 0    50   Output ~ 0
 Dig_1
-Text HLabel 5350 2650 0    50   Input ~ 0
+Text HLabel 7400 2300 0    50   Input ~ 0
 Sw_0
-Text HLabel 5350 2750 0    50   Input ~ 0
+Text HLabel 7400 2400 0    50   Input ~ 0
 Sw_1
-Text HLabel 5350 2850 0    50   Input ~ 0
+Text HLabel 7400 2500 0    50   Input ~ 0
 Sw_2
-Text HLabel 5350 2950 0    50   Input ~ 0
+Text HLabel 7400 2600 0    50   Input ~ 0
 Sw_3
-Text HLabel 5350 3050 0    50   Input ~ 0
+Text HLabel 7400 2700 0    50   Input ~ 0
 Sw_4
-Text HLabel 5350 3150 0    50   Input ~ 0
+Text HLabel 7400 2800 0    50   Input ~ 0
 Sw_5
-Text HLabel 5350 3250 0    50   Input ~ 0
+Text HLabel 7400 2900 0    50   Input ~ 0
 Sw_6
-Text HLabel 5350 3350 0    50   Input ~ 0
+Text HLabel 7400 3000 0    50   Input ~ 0
 Sw_7
-Text HLabel 5350 3550 0    50   Input ~ 0
+Text HLabel 7400 3200 0    50   Input ~ 0
 UserBtn
-Text HLabel 5350 3750 0    50   Output ~ 0
+Text HLabel 7400 3400 0    50   Output ~ 0
 Heartbeat
-Text HLabel 5350 3850 0    50   Output ~ 0
+Text HLabel 7400 3500 0    50   Output ~ 0
 UserLED
+$Comp
+L Connector:Conn_ST_STDC14 J2
+U 1 1 611C65B7
+P 8100 5200
+F 0 "J2" H 7656 5246 50  0000 R CNN
+F 1 "Conn_ST_STDC14" H 7656 5155 50  0000 R CNN
+F 2 "" H 8100 5200 50  0001 C CNN
+F 3 "https://www.st.com/content/ccc/resource/technical/document/user_manual/group1/99/49/91/b6/b2/3a/46/e5/DM00526767/files/DM00526767.pdf/jcr:content/translations/en.DM00526767.pdf" V 7750 3950 50  0001 C CNN
+	1    8100 5200
+	-1   0    0    -1
+$EndComp
+Text Label 7100 5700 0    50   ~ 0
+dbg_UART_Tx
+Text Label 7100 5600 0    50   ~ 0
+dbg_UART_Rx
+Wire Wire Line
+	7100 5600 7600 5600
+Wire Wire Line
+	7600 5700 7100 5700
+NoConn ~ 7600 5200
+NoConn ~ 7600 5400
+Text Label 7100 5000 0    50   ~ 0
+dbg_SWDIO
+Text Label 7100 4900 0    50   ~ 0
+dbg_SWCLK
+Wire Wire Line
+	7100 4900 7600 4900
+Wire Wire Line
+	7100 5000 7600 5000
+Text Label 1450 1700 0    50   ~ 0
+nRST
+Wire Wire Line
+	1450 1700 1950 1700
+Text Label 1450 2700 0    50   ~ 0
+ClkOut
+Wire Wire Line
+	1450 2700 1950 2700
+Text Label 1450 4400 0    50   ~ 0
+Boot0
+Wire Wire Line
+	1450 4400 1950 4400
+Wire Wire Line
+	3950 1900 4450 1900
+Wire Wire Line
+	3950 2000 4450 2000
+Wire Wire Line
+	3950 5700 4450 5700
+Wire Wire Line
+	3950 5800 4450 5800
+Text Label 7100 4700 0    50   ~ 0
+nRST
+Wire Wire Line
+	7100 4700 7600 4700
+$Comp
+L power:+3.3V #PWR?
+U 1 1 611FDF2D
+P 8100 4500
+F 0 "#PWR?" H 8100 4350 50  0001 C CNN
+F 1 "+3.3V" H 8115 4673 50  0000 C CNN
+F 2 "" H 8100 4500 50  0001 C CNN
+F 3 "" H 8100 4500 50  0001 C CNN
+	1    8100 4500
+	1    0    0    -1
+$EndComp
+$Comp
+L power:GND #PWR?
+U 1 1 6120BE4B
+P 8100 5900
+F 0 "#PWR?" H 8100 5650 50  0001 C CNN
+F 1 "GND" H 8105 5727 50  0000 C CNN
+F 2 "" H 8100 5900 50  0001 C CNN
+F 3 "" H 8100 5900 50  0001 C CNN
+	1    8100 5900
+	1    0    0    -1
+$EndComp
+NoConn ~ 8200 5900
+Text Label 7100 5100 0    50   ~ 0
+dbg_SWO
+Wire Wire Line
+	7100 5100 7600 5100
+Text Label 1450 3900 0    50   ~ 0
+dbg_SWO
+Wire Wire Line
+	1450 3900 1950 3900
+Text Label 1450 4000 0    50   ~ 0
+UCPD_CC2
+Text Label 1450 4200 0    50   ~ 0
+UCPD_CC1
+Wire Wire Line
+	1450 4200 1950 4200
+Wire Wire Line
+	1950 4000 1450 4000
+Text Notes 700  3500 1    50   ~ 0
+No external termination needed\ndatasheet p.180
+Text HLabel 1450 3000 0    50   BiDi ~ 0
+USB_D-
+Text HLabel 1450 3100 0    50   BiDi ~ 0
+USB_D+
+Text HLabel 1450 4000 0    50   BiDi ~ 0
+USB_CC2
+Text HLabel 1450 4200 0    50   BiDi ~ 0
+USB_CC1
+Text HLabel 4450 1900 2    50   Input ~ 0
+CAN_Rx
+Text HLabel 4450 2000 2    50   Output ~ 0
+CAN_Tx
 $EndSCHEMATC

Commit message: things changed
Parts:
- renumbered C7 to C10, C13 to C11, C17 to C12, C8 to C13, C9 to C14, C10 to C15, C14 to C16, C11 to C17, C15 to C18, C6 to C7, C12 to C8, C16 to C9, FB1 to FB2, JP1 to JP3
Changed lines of the file:
@@
 $EndDescr
 $Comp
-L power:+3.3V #PWR0101
+L power:+3.3V #PWR026
 U 1 1 611AF6AF
 P 4050 1200
-F 0 "#PWR0101" H 4050 1050 50  0001 C CNN
+F 0 "#PWR026" H 4050 1050 50  0001 C CNN
 F 1 "+3.3V" V 4065 1328 50  0000 L CNN
 F 2 "" H 4050 1200 50  0001 C CNN
@@
 Connection ~ 4050 1200
 $Comp
-L power:+3.3VA #PWR0102
+L power:+3.3VA #PWR027
 U 1 1 611B18C1
 P 4050 1400
-F 0 "#PWR0102" H 4050 1250 50  0001 C CNN
+F 0 "#PWR027" H 4050 1250 50  0001 C CNN
 F 1 "+3.3VA" V 4065 1528 50  0000 L CNN
 F 2 "" H 4050 1400 50  0001 C CNN
@@
 	4050 1500 3950 1500
 $Comp
-L Device:C_Small C6
+L Device:C_Small C7
 U 1 1 611C3A12
 P 8650 900
-F 0 "C6" H 8750 950 50  0000 L CNN
+F 0 "C7" H 8750 950 50  0000 L CNN
 F 1 "100n" H 8750 850 50  0000 L CNN
 F 2 "Capacitor_SMD:C_0805_2012Metric" H 8650 900 50  0001 C CNN
@@
 $EndComp
 $Comp
-L Device:C_Small C7
+L Device:C_Small C10
 U 1 1 611C3B82
 P 9050 900
-F 0 "C7" H 9150 950 50  0000 L CNN
+F 0 "C10" H 9150 950 50  0000 L CNN
 F 1 "100n" H 9150 850 50  0000 L CNN
 F 2 "Capacitor_SMD:C_0805_2012Metric" H 9050 900 50  0001 C CNN
@@
 $EndComp
 $Comp
-L Device:C_Small C8
+L Device:C_Small C13
 U 1 1 611C3CD6
 P 9450 900
-F 0 "C8" H 9550 950 50  0000 L CNN
+F 0 "C13" H 9550 950 50  0000 L CNN
 F 1 "100n" H 9550 850 50  0000 L CNN
 F 2 "Capacitor_SMD:C_0805_2012Metric" H 9450 900 50  0001 C CNN
@@
 $EndComp
 $Comp
-L Device:C_Small C9
+L Device:C_Small C14
 U 1 1 611C3E2A
 P 9850 900
-F 0 "C9" H 9950 950 50  0000 L CNN
+F 0 "C14" H 9950 950 50  0000 L CNN
 F 1 "100n" H 9950 850 50  0000 L CNN
 F 2 "Capacitor_SMD:C_0805_2012Metric" H 9850 900 50  0001 C CNN
@@
 $EndComp
 $Comp
-L Device:C_Small C10
+L Device:C_Small C15
 U 1 1 611C3F90
 P 10250 900
-F 0 "C10" H 10350 950 50  0000 L CNN
+F 0 "C15" H 10350 950 50  0000 L CNN
 F 1 "100n" H 10350 850 50  0000 L CNN
 F 2 "Capacitor_SMD:C_0805_2012Metric" H 10250 900 50  0001 C CNN
@@
 $EndComp
 $Comp
-L Device:C_Small C11
+L Device:C_Small C17
 U 1 1 611C40D2
 P 10750 900
-F 0 "C11" H 10850 950 50  0000 L CNN
+F 0 "C17" H 10850 950 50  0000 L CNN
 F 1 "4u7" H 10850 850 50  0000 L CNN
 F 2 "Capacitor_SMD:C_0805_2012Metric" H 10750 900 50  0001 C CNN
@@
 	10250 1000 9850 1000
 $Comp
-L power:+3.3V #PWR0103
+L power:+3.3V #PWR038
 U 1 1 611C4F25
 P 10750 800
-F 0 "#PWR0103" H 10750 650 50  0001 C CNN
+F 0 "#PWR038" H 10750 650 50  0001 C CNN
 F 1 "+3.3V" H 10765 973 50  0000 C CNN
 F 2 "" H 10750 800 50  0001 C CNN
@@
 Connection ~ 10750 800
 $Comp
-L power:GND #PWR0104
+L power:GND #PWR039
 U 1 1 611C5C55
 P 10750 1000
-F 0 "#PWR0104" H 10750 750 50  0001 C CNN
+F 0 "#PWR039" H 10750 750 50  0001 C CNN
 F 1 "GND" H 10755 827 50  0000 C CNN
 F 2 "" H 10750 1000 50  0001 C CNN
@@
 Connection ~ 10750 1000
 $Comp
-L Device:C_Small C15
+L Device:C_Small C18
 U 1 1 611C6E46
 P 10750 1750
-F 0 "C15" H 10850 1800 50  0000 L CNN
+F 0 "C18" H 10850 1800 50  0000 L CNN
 F 1 "1u" H 10850 1700 50  0000 L CNN
 F 2 "Capacitor_SMD:C_0805_2012Metric" H 10750 1750 50  0001 C CNN
@@
 $EndComp
 $Comp
-L Device:C_Small C14
+L Device:C_Small C16
 U 1 1 611C70F8
 P 10250 1750
-F 0 "C14" H 10350 1800 50  0000 L CNN
+F 0 "C16" H 10350 1800 50  0000 L CNN
 F 1 "10n" H 10350 1700 50  0000 L CNN
 F 2 "Capacitor_SMD:C_0805_2012Metric" H 10250 1750 50  0001 C CNN
@@
 $EndComp
 $Comp
-L power:+3.3VA #PWR0105
+L power:+3.3VA #PWR040
 U 1 1 611C8A81
 P 10750 1650
-F 0 "#PWR0105" H 10750 1500 50  0001 C CNN
+F 0 "#PWR040" H 10750 1500 50  0001 C CNN
 F 1 "+3.3VA" H 10765 1823 50  0000 C CNN
 F 2 "" H 10750 1650 50  0001 C CNN
@@
 	10250 1850 10750 1850
 $Comp
-L power:GNDA #PWR0106
+L power:GNDA #PWR041
 U 1 1 611D47B0
 P 10750 1850
-F 0 "#PWR0106" H 10750 1600 50  0001 C CNN
+F 0 "#PWR041" H 10750 1600 50  0001 C CNN
 F 1 "GNDA" H 10755 1677 50  0000 C CNN
 F 2 "" H 10750 1850 50  0001 C CNN
@@
 Connection ~ 10750 1850
 $Comp
-L power:GNDA #PWR0107
+L power:GNDA #PWR029
 U 1 1 611D5580
 P 4050 6900
-F 0 "#PWR0107" H 4050 6650 50  0001 C CNN
+F 0 "#PWR029" H 4050 6650 50  0001 C CNN
 F 1 "GNDA" V 4055 6772 50  0000 R CNN
 F 2 "" H 4050 6900 50  0001 C CNN
@@
 $EndComp
 $Comp
-L power:GND #PWR0108
+L power:GND #PWR030
 U 1 1 611D5916
 P 4050 7000
-F 0 "#PWR0108" H 4050 6750 50  0001 C CNN
+F 0 "#PWR030" H 4050 6750 50  0001 C CNN
 F 1 "GND" V 4055 6872 50  0000 R CNN
 F 2 "" H 4050 7000 50  0001 C CNN
@@
 	4050 6900 3950 6900
 $Comp
-L Device:C_Small C12
+L Device:C_Small C8
 U 1 1 611DA83B
 P 8650 1750
-F 0 "C12" H 8750 1800 50  0000 L CNN
+F 0 "C8" H 8750 1800 50  0000 L CNN
 F 1 "1u" H 8750 1700 50  0000 L CNN
 F 2 "Capacitor_SMD:C_0805_2012Metric" H 8650 1750 50  0001 C CNN
@@
 $EndComp
 $Comp
-L Device:C_Small C13
+L Device:C_Small C11
 U 1 1 611DA841
 P 9150 1750
-F 0 "C13" H 9250 1800 50  0000 L CNN
+F 0 "C11" H 9250 1800 50  0000 L CNN
 F 1 "10n" H 9250 1700 50  0000 L CNN
 F 2 "Capacitor_SMD:C_0805_2012Metric" H 9150 1750 50  0001 C CNN
@@
 Connection ~ 9150 1650
 $Comp
-L Jumper:Jumper_2_Bridged JP1
+L Jumper:Jumper_2_Bridged JP3
 U 1 1 611DEC2C
 P 9700 1650
-F 0 "JP1" H 9700 1753 50  0000 C CNN
+F 0 "JP3" H 9700 1753 50  0000 C CNN
 F 1 "Jumper_2_Bridged" H 9700 1754 50  0001 C CNN
 F 2 "Jumper:SolderJumper-2_P1.3mm_Bridged_RoundedPad1.0x1.5mm" H 9700 1650 50  0001 C CNN
@@
 dbg_SWCLK
 $Comp
-L power:+3.3V #PWR0111
+L power:+3.3V #PWR036
 U 1 1 611C4761
 P 9950 2600
-F 0 "#PWR0111" H 9950 2450 50  0001 C CNN
+F 0 "#PWR036" H 9950 2450 50  0001 C CNN
 F 1 "+3.3V" H 9965 2773 50  0000 C CNN
 F 2 "" H 9950 2600 50  0001 C CNN
@@
 $EndComp
 $Comp
-L power:+3.3VA #PWR0112
+L power:+3.3VA #PWR042
 U 1 1 611C4767
 P 10750 2600
-F 0 "#PWR0112" H 10750 2450 50  0001 C CNN
+F 0 "#PWR042" H 10750 2450 50  0001 C CNN
 F 1 "+3.3VA" H 10765 2773 50  0000 C CNN
 F 2 "" H 10750 2600 50  0001 C CNN
@@
 $EndComp
 $Comp
-L Device:Ferrite_Bead_Small FB1
+L Device:Ferrite_Bead_Small FB2
 U 1 1 611C476D
 P 10350 2650
-F 0 "FB1" V 10113 2650 50  0000 C CNN
+F 0 "FB2" V 10113 2650 50  0000 C CNN
 F 1 "1k@100MHz" V 10204 2650 50  0000 C CNN
 F 2 "Inductor_SMD:L_0805_2012Metric" V 10280 2650 50  0001 C CNN
@@
 $EndComp
 $Comp
-L power:GND #PWR0113
+L power:GND #PWR037
 U 1 1 611C651B
 P 9950 2900
-F 0 "#PWR0113" H 9950 2650 50  0001 C CNN
+F 0 "#PWR037" H 9950 2650 50  0001 C CNN
 F 1 "GND" H 9955 2727 50  0000 C CNN
 F 2 "" H 9950 2900 50  0001 C CNN
@@
 $EndComp
 $Comp
-L power:GNDA #PWR0114
+L power:GNDA #PWR043
 U 1 1 611C6521
 P 10750 2900
-F 0 "#PWR0114" H 10750 2650 50  0001 C CNN
+F 0 "#PWR043" H 10750 2650 50  0001 C CNN
 F 1 "GNDA" H 10755 2727 50  0000 C CNN
 F 2 "" H 10750 2900 50  0001 C CNN
@@
 $EndComp
 $Comp
-L Device:C_Small C16
+L Device:C_Small C9
 U 1 1 6121405B
 P 8850 2850
-F 0 "C16" H 8950 2900 50  0000 L CNN
+F 0 "C9" H 8950 2900 50  0000 L CNN
 F 1 "TBD" H 8950 2800 50  0000 L CNN
 F 2 "Capacitor_SMD:C_0805_2012Metric" H 8850 2850 50  0001 C CNN
@@
 	8950 2750 8850 2750
 $Comp
-L power:GND #PWR0115
+L power:GND #PWR035
 U 1 1 61216B8C
 P 9050 2950
-F 0 "#PWR0115" H 9050 2700 50  0001 C CNN
+F 0 "#PWR035" H 9050 2700 50  0001 C CNN
 F 1 "GND" H 9055 2777 50  0000 C CNN
 F 2 "" H 9050 2950 50  0001 C CNN
@@
 	9050 2850 9050 2950
 $Comp
-L power:GND #PWR0116
+L power:GND #PWR034
 U 1 1 6121C3E3
 P 9050 2550
-F 0 "#PWR0116" H 9050 2300 50  0001 C CNN
+F 0 "#PWR034" H 9050 2300 50  0001 C CNN
 F 1 "GND" H 9055 2377 50  0000 C CNN
 F 2 "" H 9050 2550 50  0001 C CNN
@@
 	8850 2950 9050 2950
 $Comp
-L Device:C_Small C17
+L Device:C_Small C12
 U 1 1 6122185F
 P 9250 2850
-F 0 "C17" H 9350 2900 50  0000 L CNN
+F 0 "C12" H 9350 2900 50  0000 L CNN
 F 1 "TBD" H 9350 2800 50  0000 L CNN
 F 2 "Capacitor_SMD:C_0805_2012Metric" H 9250 2850 50  0001 C CNN
@@
 USART1
 $Comp
-L vref:+VREF #PWR0138
+L vref:+VREF #PWR028
 U 1 1 61262CA2
 P 4050 1500
-F 0 "#PWR0138" H 4050 1350 50  0001 C CNN
+F 0 "#PWR028" H 4050 1350 50  0001 C CNN
 F 1 "+VREF" V 4065 1628 50  0000 L CNN
 F 2 "" H 4050 1500 50  0001 C CNN
@@
 $EndComp
 $Comp
-L vref:+VREF #PWR0139
+L vref:+VREF #PWR033
 U 1 1 61263302
 P 8650 1650
-F 0 "#PWR0139" H 8650 1500 50  0001 C CNN
+F 0 "#PWR033" H 8650 1500 50  0001 C CNN
 F 1 "+VREF" H 8665 1823 50  0000 C CNN
 F 2 "" H 8650 1650 50  0001 C CNN
@@
 	7100 4700 7600 4700
 $Comp
-L power:+3.3V #PWR?
+L power:+3.3V #PWR031
 U 1 1 611FDF2D
 P 8100 4500
-F 0 "#PWR?" H 8100 4350 50  0001 C CNN
+F 0 "#PWR031" H 8100 4350 50  0001 C CNN
 F 1 "+3.3V" H 8115 4673 50  0000 C CNN
 F 2 "" H 8100 4500 50  0001 C CNN
@@
 $EndComp
 $Comp
-L power:GND #PWR?
+L power:GND #PWR032
 U 1 1 6120BE4B
 P 8100 5900
-F 0 "#PWR?" H 8100 5650 50  0001 C CNN
+F 0 "#PWR032" H 8100 5650 50  0001 C CNN
 F 1 "GND" H 8105 5727 50  0000 C CNN
 F 2 "" H 8100 5900 50  0001 C CNN
