File: hardware/mcu.sch (KiCad schematic (older format))
At the start: 17 parts, among them J2 Conn_ST_STDC14, U5 STM32G474VET6, Y1 25MHz

Commit message: Changed power again
Parts:
- J2: footprint (none) -> Connector_PinHeader_1.27mm:PinHeader_2x07_P1.27mm_Vertical_SMD
Connections:
- net nRST renamed nReset
Changed lines of the file:
@@
 ClkOut
 Text HLabel 1450 1700 0    50   Input ~ 0
-nRST
+nReset
 Text Label 1450 2300 0    50   ~ 0
 ext_SPI_nSS
@@
 Text Notes 4450 1800 2    50   ~ 0
 FDCAN1
-Text HLabel 7400 1150 0    50   Output ~ 0
-Seg_0
-Text HLabel 7400 1250 0    50   Output ~ 0
-Seg_1
-Text HLabel 7400 1350 0    50   Output ~ 0
-Seg_2
-Text HLabel 7400 1450 0    50   Output ~ 0
-Seg_3
-Text HLabel 7400 1550 0    50   Output ~ 0
-Seg_4
-Text HLabel 7400 1650 0    50   Output ~ 0
-Seg_5
-Text HLabel 7400 1750 0    50   Output ~ 0
-Seg_6
-Text HLabel 7400 1850 0    50   Output ~ 0
-Seg_7
-Text HLabel 7400 1950 0    50   Output ~ 0
-Dig_0
-Text HLabel 7400 2050 0    50   Output ~ 0
-Dig_1
-Text HLabel 7400 2300 0    50   Input ~ 0
-Sw_0
-Text HLabel 7400 2400 0    50   Input ~ 0
-Sw_1
-Text HLabel 7400 2500 0    50   Input ~ 0
-Sw_2
-Text HLabel 7400 2600 0    50   Input ~ 0
-Sw_3
-Text HLabel 7400 2700 0    50   Input ~ 0
-Sw_4
-Text HLabel 7400 2800 0    50   Input ~ 0
-Sw_5
-Text HLabel 7400 2900 0    50   Input ~ 0
-Sw_6
-Text HLabel 7400 3000 0    50   Input ~ 0
-Sw_7
 Text HLabel 7400 3200 0    50   Input ~ 0
 UserBtn
@@
 F 0 "J2" H 7656 5246 50  0000 R CNN
 F 1 "Conn_ST_STDC14" H 7656 5155 50  0000 R CNN
-F 2 "" H 8100 5200 50  0001 C CNN
+F 2 "Connector_PinHeader_1.27mm:PinHeader_2x07_P1.27mm_Vertical_SMD" H 8100 5200 50  0001 C CNN
 F 3 "https://www.st.com/content/ccc/resource/technical/document/user_manual/group1/99/49/91/b6/b2/3a/46/e5/DM00526767/files/DM00526767.pdf/jcr:content/translations/en.DM00526767.pdf" V 7750 3950 50  0001 C CNN
 	1    8100 5200
@@
 Text HLabel 4450 2000 2    50   Output ~ 0
 CAN_Tx
+Text HLabel 7400 1200 0    50   Output ~ 0
+SegA
+Text HLabel 7400 1300 0    50   Output ~ 0
+SegB
+Text HLabel 7400 1400 0    50   Output ~ 0
+SegC
+Text HLabel 7400 1500 0    50   Output ~ 0
+SegD
+Text HLabel 7400 1600 0    50   Output ~ 0
+SegE
+Text HLabel 7400 1700 0    50   Output ~ 0
+SegF
+Text HLabel 7400 1800 0    50   Output ~ 0
+SegG
+Text HLabel 7400 1900 0    50   Output ~ 0
+SegDP
+Text HLabel 7400 2000 0    50   Output ~ 0
+Dig1
+Text HLabel 7400 2100 0    50   Output ~ 0
+Dig2
+Text HLabel 7400 2300 0    50   Input ~ 0
+Sw0
+Text HLabel 7400 2400 0    50   Input ~ 0
+Sw1
+Text HLabel 7400 2500 0    50   Input ~ 0
+Sw2
+Text HLabel 7400 2600 0    50   Input ~ 0
+Sw3
+Text HLabel 7400 2700 0    50   Input ~ 0
+Sw4
+Text HLabel 7400 2800 0    50   Input ~ 0
+Sw5
+Text HLabel 7400 2900 0    50   Input ~ 0
+Sw6
+Text HLabel 7400 3000 0    50   Input ~ 0
+Sw7
 $EndSCHEMATC

Commit message: Started routing
Parts:
- added J8: Conn_02x13_Odd_Even_MountingPin, Connector_IDC:IDC-Header_2x13-1MP_P2.54mm_Latch_Horizontal, symbol Connector_Generic_MountingPin:Conn_02x13_Odd_Even_MountingPin
Connections:
- net Dig1: now also U5.53 (PB14)
- net Dig2: now also U5.54 (PB15)
- net Heartbeat: now also U5.70 (PA9)
- net SegA: now also U5.55 (PD8)
- net SegB: now also U5.56 (PD9)
- net SegC: now also U5.57 (PD10)
- net SegD: now also U5.58 (PD11)
- net SegDP: now also U5.62 (PD15)
- net SegE: now also U5.59 (PD12)
- net SegF: now also U5.60 (PD13)
- net SegG: now also U5.61 (PD14)
- net Sw0: now also U5.15 (PC0)
- net Sw1: now also U5.16 (PC1)
- net Sw2: now also U5.17 (PC2)
- net Sw3: now also U5.18 (PC3)
- net Sw4: now also U5.19 (PF2)
- net Sw5: now also U5.20 (PA0)
- net Sw6: now also U5.21 (PA1)
- net Sw7: now also U5.22 (PA2)
- net UserBtn: now also U5.94 (PB7)
- net UserLED: now also U5.71 (PA10)
- net ext_CAN_Rx: now also U5.51 (PB12); no longer U5.53 (PB14)
- net SD_SPI_MISO renamed SD_MISO
- net SD_SPI_MOSI renamed SD_MOSI
- net SD_SPI_SCK renamed SD_SCK
- net SD_SPI_nSS renamed SD_nSS
Other:
- moved on the sheet: J2, U5

Commit message: things changed
Parts:
- added C?: 100n, symbol Device:C_Small
- added U?: 24AA02-OT, Package_TO_SOT_SMD:SOT-23-5, symbol Memory_EEPROM:24AA02-OT
Connections:
- net +3V3: now also C?.1, U?.4 (VCC)
- net GND: now also C?.2, U?.2 (GND)
Changed lines of the file:
@@
 Wire Wire Line
 	5250 5550 4750 5550
+$Comp
+L Memory_EEPROM:24AA02-OT U?
+U 1 1 612D8F4F
+P 6900 3700
+F 0 "U?" H 7200 4000 50  0000 R CNN
+F 1 "24AA02-OT" H 6800 4000 50  0000 R CNN
+F 2 "Package_TO_SOT_SMD:SOT-23-5" H 6900 3700 50  0001 C CNN
+F 3 "http://ww1.microchip.com/downloads/en/DeviceDoc/21709J.pdf" H 6900 3700 50  0001 C CNN
+	1    6900 3700
+	1    0    0    -1
+$EndComp
+$Comp
+L power:GND #PWR?
+U 1 1 612D94FF
+P 6900 4000
+F 0 "#PWR?" H 6900 3750 50  0001 C CNN
+F 1 "GND" H 6905 3827 50  0000 C CNN
+F 2 "" H 6900 4000 50  0001 C CNN
+F 3 "" H 6900 4000 50  0001 C CNN
+	1    6900 4000
+	1    0    0    -1
+$EndComp
+$Comp
+L power:+3.3V #PWR?
+U 1 1 612D9D14
+P 6900 3400
+F 0 "#PWR?" H 6900 3250 50  0001 C CNN
+F 1 "+3.3V" H 6915 3573 50  0000 C CNN
+F 2 "" H 6900 3400 50  0001 C CNN
+F 3 "" H 6900 3400 50  0001 C CNN
+	1    6900 3400
+	1    0    0    -1
+$EndComp
+$Comp
+L Device:C_Small C?
+U 1 1 612DA767
+P 7450 3100
+F 0 "C?" H 7542 3146 50  0000 L CNN
+F 1 "100n" H 7542 3055 50  0000 L CNN
+F 2 "" H 7450 3100 50  0001 C CNN
+F 3 "~" H 7450 3100 50  0001 C CNN
+	1    7450 3100
+	1    0    0    -1
+$EndComp
+$Comp
+L power:GND #PWR?
+U 1 1 612DB8E5
+P 7450 3200
+F 0 "#PWR?" H 7450 2950 50  0001 C CNN
+F 1 "GND" H 7455 3027 50  0000 C CNN
+F 2 "" H 7450 3200 50  0001 C CNN
+F 3 "" H 7450 3200 50  0001 C CNN
+	1    7450 3200
+	1    0    0    -1
+$EndComp
+$Comp
+L power:+3.3V #PWR?
+U 1 1 612DBB82
+P 7450 3000
+F 0 "#PWR?" H 7450 2850 50  0001 C CNN
+F 1 "+3.3V" H 7465 3173 50  0000 C CNN
+F 2 "" H 7450 3000 50  0001 C CNN
+F 3 "" H 7450 3000 50  0001 C CNN
+	1    7450 3000
+	1    0    0    -1
+$EndComp
 $EndSCHEMATC
